Commit message: 오류해결안됨

File: install/welder_moveit_config/share/welder_moveit_config/config/welder.ros2_control.xacro (robot description, xacro)
@@ -1,54 +1 @@
-<?xml version="1.0"?>
-<robot xmlns:xacro="http://www.ros.org/wiki/xacro">
-    <xacro:macro name="welder_ros2_control" params="name initial_positions_file">
-        <xacro:property name="initial_positions" value="${xacro.load_yaml(initial_positions_file)['initial_positions']}"/>
-        <ros2_control name="${name}" type="system">
-            <hardware>
-                <!-- By default, set up controllers for simulation. This won't work on real hardware -->
-                <plugin>mock_components/GenericSystem</plugin>
-            </hardware>
-            <joint name="joint_1">
-                <command_interface name="position"/>
-                <state_interface name="position">
-                  <param name="initial_value">${initial_positions['joint_1']}</param>
-                </state_interface>
-                <state_interface name="velocity"/>
-            </joint>
-            <joint name="joint_2">
-                <command_interface name="position"/>
-                <state_interface name="position">
-                  <param name="initial_value">${initial_positions['joint_2']}</param>
-                </state_interface>
-                <state_interface name="velocity"/>
-            </joint>
-            <joint name="joint_3">
-                <command_interface name="position"/>
-                <state_interface name="position">
-                  <param name="initial_value">${initial_positions['joint_3']}</param>
-                </state_interface>
-                <state_interface name="velocity"/>
-            </joint>
-            <joint name="joint_4">
-                <command_interface name="position"/>
-                <state_interface name="position">
-                  <param name="initial_value">${initial_positions['joint_4']}</param>
-                </state_interface>
-                <state_interface name="velocity"/>
-            </joint>
-            <joint name="joint_5">
-                <command_interface name="position"/>
-                <state_interface name="position">
-                  <param name="initial_value">${initial_positions['joint_5']}</param>
-                </state_interface>
-                <state_interface name="velocity"/>
-            </joint>
-            <joint name="joint_6">
-                <command_interface name="position"/>
-                <state_interface name="position">
-                  <param name="initial_value">${initial_positions['joint_6']}</param>
-                </state_interface>
-                <state_interface name="velocity"/>
-            </joint>
-        </ros2_control>
-    </xacro:macro>
-</robot>
+/home/kriso/arm_tuto_WS/src/welder_moveit_config/config/welder.ros2_control.xacro

File: install/welder_moveit_config/share/welder_moveit_config/config/welder.urdf.xacro (robot description, xacro)
@@ -1,9 +1 @@
-<?xml version="1.0"?>
-<robot xmlns:xacro="http://www.ros.org/wiki/xacro" name="welder">
-    <xacro:arg name="initial_positions_file" default="initial_positions.yaml" />
-    <!-- Import welder urdf file -->
-    <xacro:include filename="$(find welder_description)/urdf/welder.xacro" />
-    <!-- Import control_xacro -->
-    <xacro:include filename="welder.ros2_control.xacro" />
-    <xacro:welder_ros2_control name="FakeSystem" initial_positions_file="$(arg initial_positions_file)"/>
-</robot>
+/home/kriso/arm_tuto_WS/src/welder_moveit_config/config/welder.urdf.xacro

File: src/welder_description/urdf/welder.urdf (robot description, URDF)
Before this commit: robot welder, 8 links, 7 joints
Links:
- link base_link: geometry collision mesh filename=package://welder_description/meshes/base_link.stl scale=0.001 0.001 0.001; visual mesh filename=package://welder_description/meshes/base_link.stl scale=0.001 0.001 0.001
- link link_1_1: geometry collision mesh filename=package://welder_description/meshes/link_1_1.stl scale=0.001 0.001 0.001; visual mesh filename=package://welder_description/meshes/link_1_1.stl scale=0.001 0.001 0.001
- link link_2_1: geometry collision mesh filename=package://welder_description/meshes/link_2_1.stl scale=0.001 0.001 0.001; visual mesh filename=package://welder_description/meshes/link_2_1.stl scale=0.001 0.001 0.001
- link link_3_1: geometry collision mesh filename=package://welder_description/meshes/link_3_1.stl scale=0.001 0.001 0.001; visual mesh filename=package://welder_description/meshes/link_3_1.stl scale=0.001 0.001 0.001
- link link_4_1: geometry collision mesh filename=package://welder_description/meshes/link_4_1.stl scale=0.001 0.001 0.001; visual mesh filename=package://welder_description/meshes/link_4_1.stl scale=0.001 0.001 0.001
- link link_5_1: geometry collision mesh filename=package://welder_description/meshes/link_5_1.stl scale=0.001 0.001 0.001; visual mesh filename=package://welder_description/meshes/link_5_1.stl scale=0.001 0.001 0.001
- link link_6_1: geometry collision mesh filename=package://welder_description/meshes/link_6_1.stl scale=0.001 0.001 0.001; visual mesh filename=package://welder_description/meshes/link_6_1.stl scale=0.001 0.001 0.001

File: src/welder_moveit_config/config/welder.ros2_control.xacro (robot description, xacro)
@@ -6,5 +6,5 @@
             <hardware>
                 <!-- By default, set up controllers for simulation. This won't work on real hardware -->
-                <plugin>mock_components/GenericSystem</plugin>
+                <plugin>gazebo_ros2_control/GazeboSystem</plugin>
             </hardware>
             <joint name="joint_1">
@@ -51,4 +51,65 @@
             </joint>
         </ros2_control>
+        <!-- Transmissions -->
+        <transmission name="joint_1_trans">
+          <type>transmission_interface/SimpleTransmission</type>
+          <joint name="joint_1">
+            <hardwareInterface>hardware_interface/PositionJointInterface</hardwareInterface>
+          </joint>
+          <actuator name="joint_1_motor">
+            <hardwareInterface>hardware_interface/PositionJointInterface</hardwareInterface>
+            <mechanicalReduction>1</mechanicalReduction>
+          </actuator>
+        </transmission>
+        <transmission name="joint_2_trans">
+          <type>transmission_interface/SimpleTransmission</type>
+          <joint name="joint_2">
+            <hardwareInterface>hardware_interface/PositionJointInterface</hardwareInterface>
+          </joint>
+          <actuator name="joint_2_motor">
+            <hardwareInterface>hardware_interface/PositionJointInterface</hardwareInterface>
+            <mechanicalReduction>1</mechanicalReduction>
+          </actuator>
+        </transmission>
+        <transmission name="joint_3_trans">
+          <type>transmission_interface/SimpleTransmission</type>
+          <joint name="joint_3">
+            <hardwareInterface>hardware_interface/PositionJointInterface</hardwareInterface>
+          </joint>
+          <actuator name="joint_3_motor">
+            <hardwareInterface>hardware_interface/PositionJointInterface</hardwareInterface>
+            <mechanicalReduction>1</mechanicalReduction>
+          </actuator>
+        </transmission>
+        <transmission name="joint_4_trans">
+          <type>transmission_interface/SimpleTransmission</type>
+          <joint name="joint_4">
+            <hardwareInterface>hardware_interface/PositionJointInterface</hardwareInterface>
+          </joint>
+          <actuator name="joint_4_motor">
+            <hardwareInterface>hardware_interface/PositionJointInterface</hardwareInterface>
+            <mechanicalReduction>1</mechanicalReduction>
+          </actuator>
+        </transmission>
+        <transmission name="joint_5_trans">
+          <type>transmission_interface/SimpleTransmission</type>
+          <joint name="joint_5">
+            <hardwareInterface>hardware_interface/PositionJointInterface</hardwareInterface>
+          </joint>
+          <actuator name="joint_5_motor">
+            <hardwareInterface>hardware_interface/PositionJointInterface</hardwareInterface>
+            <mechanicalReduction>1</mechanicalReduction>
+          </actuator>
+        </transmission>
+        <transmission name="joint_6_trans">
+          <type>transmission_interface/SimpleTransmission</type>
+          <joint name="joint_6">
+            <hardwareInterface>hardware_interface/PositionJointInterface</hardwareInterface>
+          </joint>
+          <actuator name="joint_6_motor">
+            <hardwareInterface>hardware_interface/PositionJointInterface</hardwareInterface>
+            <mechanicalReduction>1</mechanicalReduction>
+          </actuator>
+        </transmission>
     </xacro:macro>
 </robot>

File: src/welder_moveit_config/config/welder.urdf.xacro (robot description, xacro)
@@ -2,8 +2,181 @@
 <robot xmlns:xacro="http://www.ros.org/wiki/xacro" name="welder">
     <xacro:arg name="initial_positions_file" default="initial_positions.yaml" />
-    <!-- Import welder urdf file -->
-    <xacro:include filename="$(find welder_description)/urdf/welder.xacro" />
     <!-- Import control_xacro -->
     <xacro:include filename="welder.ros2_control.xacro" />
-    <xacro:welder_ros2_control name="FakeSystem" initial_positions_file="$(arg initial_positions_file)"/>
+<link name="world">
+</link>
+<link name="base_link">
+  <inertial>
+    <origin xyz="-7.16285389829585e-11 -1.5064593165281103e-11 0.019107627086653742" rpy="0 0 0"/>
+    <mass value="2.955437891841375"/>
+    <inertia ixx="0.002819" iyy="0.002819" izz="0.004764" ixy="-0.0" iyz="-0.0" ixz="-0.0"/>
+  </inertial>
+  <visual>
+    <origin xyz="0 0 0" rpy="0 0 0"/>
+    <geometry>
+      <mesh filename="file:///home/kriso/arm_tuto_WS/src/welder_description/meshes/base_link.stl"/>
+    </geometry>
+  </visual>
+  <collision>
+    <origin xyz="0 0 0" rpy="0 0 0"/>
+    <geometry>
+      <mesh filename="file:///home/kriso/arm_tuto_WS/src/welder_description/meshes/base_link.stl"/>
+    </geometry>
+  </collision>
+</link>
+<link name="link_1_1">
+  <inertial>
+    <origin xyz="0.0 0.0009431909165482249 0.11440920058437602" rpy="0 0 0"/>
+    <mass value="2.2877730999420254"/>
+    <inertia ixx="0.009859" iyy="0.009807" izz="0.000515" ixy="0.0" iyz="-0.000185" ixz="0.0"/>
+  </inertial>
+  <visual>
+    <origin xyz="-0.0 -0.0 -0.05" rpy="0 0 0"/>
+    <geometry>
+      <mesh filename="file:///home/kriso/arm_tuto_WS/src/welder_description/meshes/link_1_1.stl"/>
+    </geometry>
+  </visual>
+  <collision>
+    <origin xyz="-0.0 -0.0 -0.05" rpy="0 0 0"/>
+    <geometry>
+      <mesh filename="file:///home/kriso/arm_tuto_WS/src/welder_description/meshes/link_1_1.stl"/>
+    </geometry>
+  </collision>
+</link>
+<link name="link_2_1">
+  <inertial>
+    <origin xyz="0.0 -0.02834196834303381 -0.012543410312423592" rpy="0 0 0"/>
+    <mass value="0.8650806084810733"/>
+    <inertia ixx="0.000478" iyy="0.0004" izz="0.000257" ixy="0.0" iyz="-1.8e-05" ixz="0.0"/>
+  </inertial>
+  <visual>
+    <origin xyz="-0.0 0.02 -0.25" rpy="0 0 0"/>
+    <geometry>
+      <mesh filename="file:///home/kriso/arm_tuto_WS/src/welder_description/meshes/link_2_1.stl"/>
+    </geometry>
+  </visual>
+  <collision>
+    <origin xyz="-0.0 0.02 -0.25" rpy="0 0 0"/>
+    <geometry>
+      <mesh filename="file:///home/kriso/arm_tuto_WS/src/welder_description/meshes/link_2_1.stl"/>
+    </geometry>
+  </collision>
+</link>
+<link name="link_3_1">
+  <inertial>
+    <origin xyz="0.0 -0.0009734727614764405 -0.056920756556270824" rpy="0 0 0"/>
+    <mass value="1.1630985552142648"/>
+    <inertia ixx="0.001298" iyy="0.00127" izz="0.000267" ixy="0.0" iyz="-3.8e-05" ixz="0.0"/>
+  </inertial>
+  <visual>
+    <origin xyz="-0.0 0.05 -0.2" rpy="0 0 0"/>
+    <geometry>
+      <mesh filename="file:///home/kriso/arm_tuto_WS/src/welder_description/meshes/link_3_1.stl"/>
+    </geometry>
+  </visual>
+  <collision>
+    <origin xyz="-0.0 0.05 -0.2" rpy="0 0 0"/>
+    <geometry>
+      <mesh filename="file:///home/kriso/arm_tuto_WS/src/welder_description/meshes/link_3_1.stl"/>
+    </geometry>
+  </collision>
+</link>
+<link name="link_4_1">
+  <inertial>
+    <origin xyz="0.0 -0.024901368509315194 0.031832335951871196" rpy="0 0 0"/>
+    <mass value="1.2085805984841382"/>
+    <inertia ixx="0.001374" iyy="0.001327" izz="0.000295" ixy="0.0" iyz="4e-06" ixz="0.0"/>
+  </inertial>
+  <visual>
+    <origin xyz="-0.0 0.075 -0.11" rpy="0 0 0"/>
+    <geometry>
+      <mesh filename="file:///home/kriso/arm_tuto_WS/src/welder_description/meshes/link_4_1.stl"/>
+    </geometry>
+  </visual>
+  <collision>
+    <origin xyz="-0.0 0.075 -0.11" rpy="0 0 0"/>
+    <geometry>
+      <mesh filename="file:///home/kriso/arm_tuto_WS/src/welder_description/meshes/link_4_1.stl"/>
+    </geometry>
+  </collision>
+</link>
+<link name="link_5_1">
+  <inertial>
+    <origin xyz="0.0 -4.404769588479962e-05 0.03489668781804081" rpy="0 0 0"/>
+    <mass value="0.7187100595069817"/>
+    <inertia ixx="0.000352" iyy="0.000343" izz="0.000159" ixy="-0.0" iyz="1e-06" ixz="0.0"/>
+  </inertial>
+  <visual>
+    <origin xyz="-0.0 0.1 -0.2" rpy="0 0 0"/>
+    <geometry>
+      <mesh filename="file:///home/kriso/arm_tuto_WS/src/welder_description/meshes/link_5_1.stl"/>
+    </geometry>
+  </visual>
+  <collision>
+    <origin xyz="-0.0 0.1 -0.2" rpy="0 0 0"/>
+    <geometry>
+      <mesh filename="file:///home/kriso/arm_tuto_WS/src/welder_description/meshes/link_5_1.stl"/>
+    </geometry>
+  </collision>
+</link>
+<link name="link_6_1">
+  <inertial>
+    <origin xyz="0.0 -0.01680268432280871 1.6653345369377348e-16" rpy="0 0 0"/>
+    <mass value="0.26501912859947435"/>
+    <inertia ixx="5.2e-05" iyy="3.9e-05" izz="5.2e-05" ixy="0.0" iyz="-0.0" ixz="-0.0"/>
+  </inertial>
+  <visual>
+    <origin xyz="-0.0 0.12 -0.25" rpy="0 0 0"/>
+    <geometry>
+      <mesh filename="file:///home/kriso/arm_tuto_WS/src/welder_description/meshes/link_6_1.stl"/>
+    </geometry>
+  </visual>
+  <collision>
+    <origin xyz="-0.0 0.12 -0.25" rpy="0 0 0"/>
+    <geometry>
+      <mesh filename="file:///home/kriso/arm_tuto_WS/src/welder_description/meshes/link_6_1.stl"/>
+    </geometry>
+  </collision>
+</link>
+<joint name="world_joint" type="fixed">
+  <parent link="world"/>
+  <child link="base_link"/>
+</joint>
+<joint name="joint_1" type="continuous">
+  <origin xyz="0.0 0.0 0.05" rpy="0 0 0"/>
+  <parent link="base_link"/>
+  <child link="link_1_1"/>
+  <axis xyz="0.0 0.0 1.0"/>
+</joint>
+<joint name="joint_2" type="continuous">
+  <origin xyz="0.0 -0.02 0.2" rpy="0 0 0"/>
+  <parent link="link_1_1"/>
+  <child link="link_2_1"/>
+  <axis xyz="0.0 -1.0 0.0"/>
+</joint>
+<joint name="joint_3" type="continuous">
+  <origin xyz="0.0 -0.03 -0.05" rpy="0 0 0"/>
+  <parent link="link_2_1"/>
+  <child link="link_3_1"/>
+  <axis xyz="0.0 0.0 -1.0"/>
+</joint>
+<joint name="joint_4" type="continuous">
+  <origin xyz="0.0 -0.025 -0.09" rpy="0 0 0"/>
+  <parent link="link_3_1"/>
+  <child link="link_4_1"/>
+  <axis xyz="0.0 1.0 0.0"/>
+</joint>
+<joint name="joint_5" type="continuous">
+  <origin xyz="0.0 -0.025 0.09" rpy="0 0 0"/>
+  <parent link="link_4_1"/>
+  <child link="link_5_1"/>
+  <axis xyz="0.0 0.0 1.0"/>
+</joint>
+<joint name="joint_6" type="continuous">
+  <origin xyz="0.0 -0.02 0.05" rpy="0 0 0"/>
+  <parent link="link_5_1"/>
+  <child link="link_6_1"/>
+  <axis xyz="0.0 -1.0 0.0"/>
+</joint>
+    <xacro:welder_ros2_control name="WelderSystem" initial_positions_file="$(arg initial_positions_file)"/>
 </robot>
